Commit message: dev: implement a demo launch file that supports IRL realsense cams and declares a "simulation" arg

File: src/kalman/urdf/kalman.urdf.xacro (robot description, xacro)
@@ -1,17 +1,27 @@
+<!-- This Xacro file is used to generate an URDF description of the Kalman robot.
+The description defines all the TF nodes that are children of base_link. -->
 <?xml version="1.0"?>
 <robot xmlns:xacro="http://www.ros.org/wiki/xacro" name="kalman">
     <xacro:include filename="$(find realsense2_description)/urdf/_d455.urdf.xacro" />
     <link name="base_link" />
-    <xacro:sensor_d455 name="d455_front" parent="base_link" use_nominal_extrinsics="true">>
+    <xacro:sensor_d455 name="d455_front" parent="base_link" use_nominal_extrinsics="true">
         <origin xyz="1 0 0" rpy="0 0 0"/>
     </xacro:sensor_d455>
-    <xacro:sensor_d455 name="d455_back" parent="base_link" use_nominal_extrinsics="true">>
-        <origin xyz="-1 0 0" rpy="0 0 0"/>
+    <xacro:sensor_d455 name="d455_back" parent="base_link" use_nominal_extrinsics="true">
+        <origin xyz="-1 0 0" rpy="0 0 3.141592654"/>
     </xacro:sensor_d455>
-    <xacro:sensor_d455 name="d455_left" parent="base_link" use_nominal_extrinsics="true">>
-        <origin xyz="0 1 0" rpy="0 0 0"/>
+    <xacro:sensor_d455 name="d455_left" parent="base_link" use_nominal_extrinsics="true">
+        <origin xyz="0 1 0" rpy="0 0 1.570796327"/>
     </xacro:sensor_d455>
-    <xacro:sensor_d455 name="d455_right" parent="base_link" use_nominal_extrinsics="true">>
-        <origin xyz="0 -1 0" rpy="0 0 0"/>
+    <xacro:sensor_d455 name="d455_right" parent="base_link" use_nominal_extrinsics="true">
+        <origin xyz="0 -1 0" rpy="0 0 -1.570796327"/>
     </xacro:sensor_d455>
+    <!-- <gazebo>
+    <plugin name="my_rgbd_camera" filename="libignition_sensors7_rgbd_camera_dev.so">
+      <alwaysOn>true</alwaysOn>
+      <updateRate>10.0</updateRate>
+      <cameraName>rgbd_camera</cameraName>
+      Other camera parameters
+    </plugin> -->
+  <!-- </gazebo> -->
 </robot>
