Commit message: feat: robot_localization using just IMU (yes, it does drift away); dev: move urdfs to config folder

File: src/kalman/config/kalman.urdf.xacro (robot description, xacro)
@@ -5,15 +5,29 @@
     <xacro:include filename="$(find realsense2_description)/urdf/_d455.urdf.xacro" />
     <link name="base_link" />
+    <!-- IMU -->
+    <link name="imu_link" >
+        <inertial>
+                <mass value="0.001"/>
+                <origin rpy="0 0 0" xyz="0 0 0"/>
+                <inertia ixx="0.0001" ixy="0" ixz="0" iyy="0.000001" iyz="0" izz="0.0001"/>
+            </inertial>
+    </link>
+    <joint name="imu_joint" type="fixed">
+        <origin xyz="0.3 0 -0.01"/>
+        <parent link="base_link"/>
+        <child link="imu_link"/>
+    </joint>
+    <!-- RealSense -->
     <xacro:sensor_d455 name="d455_front" parent="base_link" use_nominal_extrinsics="true">
-        <origin xyz="1 0 0" rpy="0 0 0"/>
+        <origin xyz="0.32 0.115 0.21" rpy="0 0 0" />
     </xacro:sensor_d455>
     <xacro:sensor_d455 name="d455_back" parent="base_link" use_nominal_extrinsics="true">
-        <origin xyz="-1 0 0" rpy="0 0 3.141592654"/>
+        <origin xyz="-0.36 -0.195 0.25" rpy="0 0 -3.14" />
     </xacro:sensor_d455>
     <xacro:sensor_d455 name="d455_left" parent="base_link" use_nominal_extrinsics="true">
-        <origin xyz="0 1 0" rpy="0 0 1.570796327"/>
+        <origin xyz="0.29 0.145 0.28" rpy="0 0 1.57" />
     </xacro:sensor_d455>
     <xacro:sensor_d455 name="d455_right" parent="base_link" use_nominal_extrinsics="true">
-        <origin xyz="0 -1 0" rpy="0 0 -1.570796327"/>
+        <origin xyz="-0.33 -0.225 0.33" rpy="0 0 -1.57" />
     </xacro:sensor_d455>
 </robot>

Commit message: feat: altimeter; dev: some experiments with nav2 (nothing works yet)

File: src/kalman/config/kalman.urdf.xacro (robot description, xacro)
@@ -31,3 +31,16 @@
         <origin xyz="-0.33 -0.225 0.33" rpy="0 0 -1.57" />
     </xacro:sensor_d455>
+    <!-- Altimeter -->
+    <link name="altimeter_link" >
+        <inertial>
+                <mass value="0.001"/>
+                <origin rpy="0 0 0" xyz="0 0 0"/>
+                <inertia ixx="0.0001" ixy="0" ixz="0" iyy="0.000001" iyz="0" izz="0.0001"/>
+            </inertial>
+    </link>
+    <joint name="altimeter_joint" type="fixed">
+        <origin xyz="0.3 0 -0.01"/>
+        <parent link="base_link"/>
+        <child link="altimeter_link"/>
+    </joint>
 </robot>
